File: AT-sound/AT-sound/_autosave-AT-sound.sch (KiCad schematic (older format))
At the start: 8 parts

Commit message: starred
Connections:
- wire segments 14 -> 15
Other:
- moved on the sheet: C?, R?
Changed lines of the file:
@@
 L Device:C C?
 U 1 1 6094155F
-P 6300 2750
-F 0 "C?" H 6415 2796 50  0000 L CNN
-F 1 "C" H 6415 2705 50  0000 L CNN
-F 2 "Capacitor_SMD:C_0805_2012Metric" H 6338 2600 50  0001 C CNN
-F 3 "~" H 6300 2750 50  0001 C CNN
-	1    6300 2750
-	1    0    0    -1
+P 6300 3050
+F 0 "C?" H 6415 3096 50  0000 L CNN
+F 1 "C" H 6415 3005 50  0000 L CNN
+F 2 "Capacitor_SMD:C_0805_2012Metric" H 6338 2900 50  0001 C CNN
+F 3 "~" H 6300 3050 50  0001 C CNN
+	1    6300 3050
+	0    1    1    0
 $EndComp
 $Comp
 L Device:R R?
 U 1 1 60941978
-P 5900 2100
-F 0 "R?" H 5970 2146 50  0000 L CNN
-F 1 "R" H 5970 2055 50  0000 L CNN
-F 2 "" V 5830 2100 50  0001 C CNN
-F 3 "~" H 5900 2100 50  0001 C CNN
-	1    5900 2100
+P 5800 3350
+F 0 "R?" H 5870 3396 50  0000 L CNN
+F 1 "R" H 5870 3305 50  0000 L CNN
+F 2 "" V 5730 3350 50  0001 C CNN
+F 3 "~" H 5800 3350 50  0001 C CNN
+	1    5800 3350
 	1    0    0    -1
 $EndComp
@@
 L Device:R R?
 U 1 1 60941C44
-P 5900 2600
-F 0 "R?" H 5970 2646 50  0000 L CNN
-F 1 "R" H 5970 2555 50  0000 L CNN
-F 2 "" V 5830 2600 50  0001 C CNN
-F 3 "~" H 5900 2600 50  0001 C CNN
-	1    5900 2600
+P 5800 3850
+F 0 "R?" H 5870 3896 50  0000 L CNN
+F 1 "R" H 5870 3805 50  0000 L CNN
+F 2 "" V 5730 3850 50  0001 C CNN
+F 3 "~" H 5800 3850 50  0001 C CNN
+	1    5800 3850
 	1    0    0    -1
 $EndComp
@@
 Wire Wire Line
 	3350 5900 3750 5900
+Text GLabel 3800 2500 2    50   Input ~ 0
+Relay
+Wire Wire Line
+	7100 1950 7100 4250
 $EndSCHEMATC
