File: AT-sound/AT-sound/AT-sound.kicad_pcb (KiCad board)
At the start: 2 copper layers, 17.6 x 17.6 mm, 25 parts, among them J1 PWR, J2 Sound OUT, J3 Sound IN, Q1 AQY212S, U1 ATtiny24-20SSU, U2 SFH617A-2X006, U3 SFH617A-2X006

Commit message: finished routing, questioning its existance
Parts:
- added TP7: RELAY, TestPoint:TestPoint_Pad_D1.0mm, F.Cu at (163.8, 63.3)
- moved REF** 13.3 mm to (164.6, 75.4)
Routing:
- net (no net): track 13.1 -> 0.00 mm
- net GND: track 53.5 -> 60.4 mm
- net Relay: track 8.18 -> 13.2 mm
Other:
- board text removed: "RG"
