File: AT-sound/AT-sound/AT-sound.sch (KiCad schematic (older format))
At the start: 8 parts

Commit message: finished routing
Parts:
- removed D?: DIODE, symbol pspice:DIODE
- removed K?: AZ850-x, Relay_THT:Relay_DPDT_FRT5, symbol Relay:AZ850-x
- removed Q?: 2N7000, Package_TO_SOT_THT:TO-92_Inline, symbol Transistor_FET:2N7000
- added C3: 0.22uF, Capacitor_SMD:C_0805_2012Metric, symbol Device:C
- added D1, D2: DZ2S150X0L, Diode_SMD:D_SOD-523, symbol Diode:DZ2S150X0L
- added J1: PWR, Connector_PinSocket_2.54mm:PinSocket_1x02_P2.54mm_Vertical, symbol Connector:Conn_01x02_Female
- added J2: Sound OUT, Connector_PinSocket_2.54mm:PinSocket_1x03_P2.54mm_Vertical, symbol Connector:Conn_01x03_Male
- added J3: Sound IN, Connector_PinSocket_2.54mm:PinSocket_1x03_P2.54mm_Vertical, symbol Connector:Conn_01x03_Female
- added Q1: AQY212S, Package_TO_SOT_SMD:SOT-23, symbol Device:Q_NMOS_GSD
- added R3, R4: 39K, Resistor_SMD:R_0603_1608Metric, symbol Device:R
- added R5, R6: 700r, Resistor_SMD:R_0603_1608Metric, symbol Device:R
- added TP1: 5v, TestPoint:TestPoint_Pad_D1.0mm, symbol Connector:TestPoint
- added TP2: GND, TestPoint:TestPoint_Pad_D1.0mm, symbol Connector:TestPoint
- added TP3: RESET, TestPoint:TestPoint_Pad_D1.0mm, symbol Connector:TestPoint
- added TP4: SKL, TestPoint:TestPoint_Pad_D1.0mm, symbol Connector:TestPoint
- added TP5: MISO, TestPoint:TestPoint_Pad_D1.0mm, symbol Connector:TestPoint
- added TP6: MOSI, TestPoint:TestPoint_Pad_D1.0mm, symbol Connector:TestPoint
- added U2, U3: SFH617A-2X006, Package_SO:SOP-4_3.8x4.1mm_P2.54mm, symbol Isolator:SFH617A-2X006
- C2: renamed from C?; value C -> 0.22uF
- R1, R2: renamed from R?; value R -> 39K; footprint (none) -> Resistor_SMD:R_0603_1608Metric
- gave numbers to parts that had none: 2
Connections:
- net +5V: now also R1.1, D1.1 (K), D2.1 (K), J1.2 (Pin_2), R3.1, TP1.1, U2.1, U3.1
- net GND: now also R2.2, J1.1 (Pin_1), J2.1 (Pin_1), J3.1 (Pin_1), Q1.2 (S), R4.2, TP2.1
- net Relay: now also U1.10 (PA3), Q1.1 (G)
- net Sense_L: now reaches U1.11 (PA2)
- net Sense_L: now also C3.2, D2.2 (A), R3.2, R4.1
- net Sense_R: now reaches U1.12 (PA1)
- net Sense_R: now also C2.2, R1.2, R2.1, D1.2 (A)
- net at U1.4 (~RESET~/PB3): now also TP3.1
- net at U1.7 (PA6): now also TP6.1
- net at U1.8 (PA5): now also TP5.1
- net at U1.9 (PA4): now also TP4.1
- net at C2.1: now also J3.3 (Pin_3), U2.3
- new net: C3.1, J3.2 (Pin_2), U3.3
- new net: J2.2 (Pin_2), U3.4
- new net: J2.3 (Pin_3), U2.4
- new net: R5.1, U2.2
- new net: Q1.3 (D), R5.2, R6.2
- new net: R6.1, U3.2
Other:
- note added: "opto cupler part number wrong."
- moved on the sheet: C2, R1, R2

Commit message: finished routing, questioning its existance
Parts:
- added TP7: RELAY, TestPoint:TestPoint_Pad_D1.0mm, symbol Connector:TestPoint
Connections:
- net Relay: now also TP7.1
Changed lines of the file:
@@
 Relay
 Wire Wire Line
-	5950 3750 6350 3750
+	5950 3750 6050 3750
 Text GLabel 3750 2700 2    50   Input ~ 0
 Relay
@@
 Text Notes 6550 2550 0    50   ~ 0
 opto cupler part number wrong.
+$Comp
+L Connector:TestPoint TP7
+U 1 1 609729FE
+P 6050 3750
+F 0 "TP7" H 6108 3868 50  0000 L CNN
+F 1 "RELAY" H 6108 3777 50  0000 L CNN
+F 2 "TestPoint:TestPoint_Pad_D1.0mm" H 6250 3750 50  0001 C CNN
+F 3 "~" H 6250 3750 50  0001 C CNN
+	1    6050 3750
+	1    0    0    -1
+$EndComp
+Connection ~ 6050 3750
+Wire Wire Line
+	6050 3750 6350 3750
 $EndSCHEMATC
